File: hardware/kicad/RoyalNode/RoyalNode.kicad_sch (KiCad schematic)
At the start: 0 parts

Commit message: Generate initial Rev A schematic capture
Parts:
- added F1: Littelfuse 0483002.DR, symbol RoyalNode:RN_TWO_PIN_POWER_PART
- added J1: XT30PW-M SOLAR, symbol RoyalNode:RN_XT30PW_M
- added J2: XT30PW-M BATTERY, symbol RoyalNode:RN_XT30PW_M
- added J3: XIAO BAT HARNESS, symbol RoyalNode:RN_JST_PH_2
- added J4: BATTERY NTC, symbol RoyalNode:RN_JST_PH_2
- added J5: Molex 0732511150 SMA, symbol RoyalNode:RN_SMA_EDGE
- added L1: Coilcraft XAL7070-222MEC, symbol RoyalNode:RN_TWO_PIN_POWER_PART
- added L2: Coilcraft XAL7030-222MEC, symbol RoyalNode:RN_TWO_PIN_POWER_PART
- added MOD1: XIAO nRF52840, symbol RoyalNode:RN_XIAO_nRF52840_SOCKET
- added MOD2: E22-900M33S, symbol RoyalNode:RN_E22_900M33S
- added Q1, Q2, Q3: ISA170170N04LMDS, symbol RoyalNode:RN_ISA170170N04LMDS
- added U1: BQ25798RQMR, symbol RoyalNode:RN_BQ25798RQMR
- added U2: LM66100DCKR, symbol RoyalNode:RN_LM66100DCKR
- added U3: TPS61088RHLR, symbol RoyalNode:RN_TPS61088RHLR
- added U4: LTC4365ITS8-1, symbol RoyalNode:RN_LTC4365ITS8_1
Connections:
- new net 3V3: MOD1.3V3
- new net 5V_RADIO: MOD2.10 (VCC_5V), MOD2.9 (VCC_5V), U3.14 (VOUT), U3.15 (VOUT), U3.16 (VOUT)
- new net BATP_KELVIN: U1.18 (BATP)
- new net BAT_RAW: J2.1 (PLUS), U1.22 (BAT), U1.23 (BAT), U2.1 (VIN)
- new net BOOST_BOOT: U3.8 (BOOT)
- new net BOOST_COMP: U3.18 (COMP)
- new net BOOST_EN: MOD1.D7 (D7/P1.12_BOOST_EN), U3.2 (EN)
- new net BOOST_FB: U3.17 (FB)
- new net BOOST_FSW: U3.3 (FSW)
- new net BOOST_ILIM: U3.19 (ILIM)
- new net BOOST_SS: U3.10 (SS)
- new net BOOST_SW: L2.2, U3.4 (SW), U3.5 (SW), U3.6 (SW), U3.7 (SW)
- new net BOOST_VCC: U3.1 (VCC)
- new net BQ_ACDRV1: Q2.2 (G1), Q2.4 (G2), U1.11 (ACDRV1)
- new net BQ_ACDRV2: Q3.2 (G1), Q3.4 (G2), U1.10 (ACDRV2)
- new net BQ_BTST1: U1.4 (BTST1)
- new net BQ_BTST2: U1.19 (BTST2)
- new net BQ_INT: U1.21 (INT)
- new net BQ_PMID: U1.29 (PMID)
- new net BQ_PROG: U1.20 (PROG)
- new net BQ_REGN: U1.17 (ILIM_HIZ), U1.5 (REGN)
- new net BQ_SDRV: U1.24 (SDRV)
- new net BQ_SOLAR_SELECTOR_COMMON: Q2.1 (S1), Q2.6 (S2)
- new net BQ_STAT: U1.1 (STAT)
- new net BQ_SW1: L1.1, U1.28 (SW1)
- new net BQ_SW2: L1.2, U1.26 (SW2)
- new net BQ_SYS: L2.1, U1.25 (SYS), U3.9 (VIN)
- new net BQ_TS: U1.16 (TS)
- new net BQ_USB_SELECTOR_COMMON: Q3.1 (S1), Q3.6 (S2)
- new net BQ_VBUS: Q2.3 (D2), Q2.5 (D2), Q3.3 (D2), Q3.5 (D2), U1.2 (VBUS), U1.3 (VBUS)
- new net E22_BUSY: MOD1.D2 (D2/P0.28_BUSY), MOD2.14 (BUSY)
- new net E22_DIO1: MOD1.D1 (D1/P0.03_DIO1), MOD2.13 (DIO1)
- new net E22_NRST: MOD1.D0 (D0/P0.02_NRST), MOD2.15 (NRST)
- new net E22_NSS: MOD1.D3 (D3/P0.29_NSS), MOD2.19 (NSS)
- new net E22_RXEN: MOD1.D6 (D6/P1.11_RXEN), MOD2.6 (RXEN)
- new net E22_TXEN_DIO2: MOD2.7 (TXEN), MOD2.8 (DIO2)
- new net GND: J1.2 (MINUS), J2.2 (MINUS), J3.2 (PIN2), J4.2 (PIN2), J5.2 (SHIELD), J5.3 (SHIELD), J5.4 (SHIELD), J5.5 (SHIELD), MOD1.GND, MOD2.1 (GND), MOD2.11 (GND), MOD2.12 (GND), MOD2.2 (GND), MOD2.20 (RF_GND), MOD2.22 (RF_GND), MOD2.3 (GND), MOD2.4 (GND), MOD2.5 (GND), U1.13 (CE_N), U1.27 (GND), U2.2 (GND), U2.5 (ST), U3.11 (NC_GND), U3.12 (NC_GND), U3.20 (AGND), U3.21 (PGND_EP), U4.4 (GND)
- new net I2C_SCL: MOD1.D5 (D5/P0.05_SCL), U1.14 (SCL)
- new net I2C_SDA: MOD1.D4 (D4/P0.04_SDA), U1.15 (SDA)
- new net NTC_SENSE: J4.1 (PIN1)
- new net OV_NODE: U4.3 (OV)
- new net RF_915: J5.1 (CENTER), MOD2.21 (ANT_50R)
- new net SOLAR_FUSED: F1.2, Q1.7 (D1), Q1.8 (D1), U4.1 (VIN), U4.5 (SHDN)
- new net SOLAR_PROTECTED: Q1.3 (D2), Q1.5 (D2), Q2.7 (D1), Q2.8 (D1), U1.9 (VAC1_SOLAR), U4.7 (VOUT)
- new net SOLAR_PROT_COMMON: Q1.1 (S1), Q1.6 (S2)
- new net SOLAR_PROT_GATE: Q1.2 (G1), Q1.4 (G2), U4.8 (GATE)
- new net SOLAR_RAW: F1.1, J1.1 (PLUS)
- new net SPI_MISO: MOD1.D9 (D9/P1.14_MISO), MOD2.16 (MISO)
- new net SPI_MOSI: MOD1.D10 (D10/P1.15_MOSI), MOD2.17 (MOSI)
- new net SPI_SCK: MOD1.D8 (D8/P1.13_SCK), MOD2.18 (SCK)
- new net USB_VBUS_RAW: MOD1.5V (5V/VBUS), Q3.7 (D1), Q3.8 (D1), U1.8 (VAC2_USB)
- new net UV_NODE: U4.2 (UV)
- new net XIAO_BAT_ISO: J3.1 (PIN1), U2.3 (CE), U2.6 (VOUT)
- no-connect marks 0 -> 6
Other:
- note added: "Generated Rev A capture scaffold from SCHEMATIC_CAPTURE_SEED_REV_A.csv.\nSymbols use global labels for reviewable net intent; final passives, footprints, and routed wires remain pending."
- note added: "Two-terminal power-path parts F1/L1/L2 are captured with RN_TWO_PIN_POWER_PART.\nExact fuse and inductor footprints remain pending footprint release."
- note removed: "RoyalNode Rev A schematic capture starts here. Authoritative source documents: - docs/DESIGN_FREEZE_REV_A.md - docs/NET_MAP_REV_A.md - docs/PIN_AUDIT_REV_A.md - docs/RF_DESIGN_REV_A.md Next KiCad task: create/import verified symbols and footprints, then capture the power tree, XIAO socket, E22 module, charger, 5 V boost, and RF connector sheets."

Commit message: Expand generated schematic to ERC clean capture
Parts:
- added C200, C201, C202, C203, C204, C205, C206, C207, C208, C209, C210, C211: 10 uF 50 V, symbol RoyalNode:RN_TWO_PIN_POWER_PART
- added C212, C213, C214, C404: 100 nF 50 V, symbol RoyalNode:RN_TWO_PIN_POWER_PART
- added C215: 4.7 uF 25 V, symbol RoyalNode:RN_TWO_PIN_POWER_PART
- added C216, C217: 47 nF 50 V, symbol RoyalNode:RN_TWO_PIN_POWER_PART
- added C218: 1 nF 50 V, symbol RoyalNode:RN_TWO_PIN_POWER_PART
- added C400, C401, C500, C501: 22 uF 16 V, symbol RoyalNode:RN_TWO_PIN_POWER_PART
- added C402, C403: 47 uF 10 V, symbol RoyalNode:RN_TWO_PIN_POWER_PART
- added C405: 2.2 uF, symbol RoyalNode:RN_TWO_PIN_POWER_PART
- added C406: 100 nF, symbol RoyalNode:RN_TWO_PIN_POWER_PART
- added C407: 47 nF, symbol RoyalNode:RN_TWO_PIN_POWER_PART
- added C408: 4.7 nF, symbol RoyalNode:RN_TWO_PIN_POWER_PART
- added C502: 1 uF 16 V, symbol RoyalNode:RN_TWO_PIN_POWER_PART
- added C503: 330 uF 10 V polymer, symbol RoyalNode:RN_TWO_PIN_POWER_PART
- added D1: Red 0603 LED, symbol RoyalNode:RN_TWO_PIN_POWER_PART
- added PF1, PF2, PF3, PF4, PF5, PF6: PWR_FLAG, symbol RoyalNode:RN_PWR_FLAG
- added R100: 1.87 MOhm 1%, symbol RoyalNode:RN_TWO_PIN_POWER_PART
- added R101: 104 kOhm 0.1%, symbol RoyalNode:RN_TWO_PIN_POWER_PART
- added R102: 40.2 kOhm 0.1%, symbol RoyalNode:RN_TWO_PIN_POWER_PART
- added R103, R403, R405: 100 kOhm, symbol RoyalNode:RN_TWO_PIN_POWER_PART
- added R200: 5.23 kOhm 1%, symbol RoyalNode:RN_TWO_PIN_POWER_PART
- added R201: 30.1 kOhm 1%, symbol RoyalNode:RN_TWO_PIN_POWER_PART
- added R202: 100 Ohm, symbol RoyalNode:RN_TWO_PIN_POWER_PART
- added R203: 4.70 kOhm 1%, symbol RoyalNode:RN_TWO_PIN_POWER_PART
- added R204, R205, R206: 10 kOhm, symbol RoyalNode:RN_TWO_PIN_POWER_PART
- added R207: 2.2 kOhm 1%, symbol RoyalNode:RN_TWO_PIN_POWER_PART
- added R400: 176 kOhm 0.1%, symbol RoyalNode:RN_TWO_PIN_POWER_PART
- added R401: 56.0 kOhm 0.1%, symbol RoyalNode:RN_TWO_PIN_POWER_PART
- added R402: 330 kOhm, symbol RoyalNode:RN_TWO_PIN_POWER_PART
- added R404: 20.0 kOhm, symbol RoyalNode:RN_TWO_PIN_POWER_PART
- added TH1: 10 kOhm NTC, symbol RoyalNode:RN_TWO_PIN_POWER_PART
Connections:
- net 3V3: now also D1.1, R204.1, R205.1, R206.1
- net 5V_RADIO: now also C402.1, C403.1, C500.1, C501.1, C502.1, C503.1, R400.1
- net BATP_KELVIN: now also R202.2
- net BAT_RAW: now also C210.1, C211.1, PF5.1 (PWR), R202.1
- net BOOST_BOOT: now also C406.1
- net BOOST_COMP: now also R404.1
- net BOOST_EN: now also R405.1
- net BOOST_FB: now also R400.2, R401.1
- net BOOST_FSW: now also R402.1
- net BOOST_ILIM: now also R403.1
- net BOOST_SS: now also C407.1
- net BOOST_SW: now also C406.2, R402.2
- net BOOST_VCC: now also C405.1
- net BQ_BTST1: now also C216.1
- net BQ_BTST2: now also C217.1
- net BQ_INT: now also R204.2
- net BQ_PMID: now also C202.1, C203.1, C204.1, C213.1
- net BQ_PROG: now also R203.1
- net BQ_REGN: now also C215.1, R200.1
- net BQ_SDRV: now also C218.1
- net BQ_STAT: now also R207.2
- net BQ_SW1: now also C216.2
- net BQ_SW2: now also C217.2
- net BQ_SYS: now also C205.1, C206.1, C207.1, C208.1, C209.1, C214.1, C400.1, C401.1, C404.1
- net BQ_TS: now also R200.2, R201.1
- net BQ_VBUS: now also C200.1, C201.1, C212.1, PF6.1 (PWR)
- net GND: now also C200.2, C201.2, C202.2, C203.2, C204.2, C205.2, C206.2, C207.2, C208.2, C209.2, C210.2, C211.2, C212.2, C213.2, C214.2, C215.2, C218.2, C400.2, C401.2, C402.2, C403.2, C404.2, C405.2, C407.2, C408.2, C500.2, C501.2, C502.2, C503.2, PF1.1 (PWR), R102.2, R203.2, R401.2, R403.2, R405.2, TH1.2
- net I2C_SCL: now also R206.2
- net I2C_SDA: now also R205.2
- net NTC_SENSE: now also R201.2, TH1.1
- net OV_NODE: now also R101.2, R102.1
- net SOLAR_FUSED: now also PF3.1 (PWR), R100.1, R103.1; no longer U4.5 (SHDN)
- net SOLAR_PROTECTED: now also PF4.1 (PWR)
- net USB_VBUS_RAW: now also PF2.1 (PWR)
- net UV_NODE: now also R100.2, R101.1
- new net BOOST_COMP_RC: C408.1, R404.2
- new net CHG_LED_K: D1.2, R207.1
- new net LTC_SHDN: R103.2, U4.5 (SHDN)
Other:
- note added: "Two-terminal power-path parts and support passives are captured with RN_TWO_PIN_POWER_PART.\nExact passive footprints remain pending footprint release and layout review."
- note removed: "Two-terminal power-path parts F1/L1/L2 are captured with RN_TWO_PIN_POWER_PART.\nExact fuse and inductor footprints remain pending footprint release."

Commit message: Assign major schematic footprints
Parts:
- J1, J2: footprint (none) -> RoyalNode:J_POWER_XT30PW_M_C431092_RC
- L1: footprint (none) -> RoyalNode:L1_COILCRAFT_XAL7070_222MEC_RC
- L2: footprint (none) -> RoyalNode:L2_COILCRAFT_XAL7030_222MEC_RC
- MOD1: footprint (none) -> RoyalNode:MOD1_XIAO_NRF52840_SOCKET_C53202181_RC
- MOD2: footprint (none) -> RoyalNode:MOD2_E22_900M33S_JLC_C22399506_RC
- Q1, Q2, Q3: footprint (none) -> RoyalNode:Q_POWER_INFINEON_PG_DSO_8_27_RC
- U1: footprint (none) -> RoyalNode:U1_BQ25798_RQM0029A_RC
- U2: footprint (none) -> RoyalNode:U2_LM66100_DCK0006A_SC70_6_RC
- U3: footprint (none) -> RoyalNode:U3_TPS61088_RHL0020A_THERMALVIAS_RC
- U4: footprint (none) -> RoyalNode:U4_LTC4365_TSOT23_8_RC
Changed lines of the file:
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@@
       )
     )
-    (property "Footprint" ""
+    (property "Footprint" "RoyalNode:MOD1_XIAO_NRF52840_SOCKET_C53202181_RC"
       (at 55.88 66.04 0)
       (effects
@@
       )
     )
-    (property "Footprint" ""
+    (property "Footprint" "RoyalNode:MOD2_E22_900M33S_JLC_C22399506_RC"
       (at 55.88 127.00 0)
       (effects
@@
       )
     )
-    (property "Footprint" ""
+    (property "Footprint" "RoyalNode:U1_BQ25798_RQM0029A_RC"
       (at 149.86 69.85 0)
       (effects
@@
       )
     )
-    (property "Footprint" ""
+    (property "Footprint" "RoyalNode:U2_LM66100_DCK0006A_SC70_6_RC"
       (at 248.92 41.91 0)
       (effects
@@
       )
     )
-    (property "Footprint" ""
+    (property "Footprint" "RoyalNode:U3_TPS61088_RHL0020A_THERMALVIAS_RC"
       (at 248.92 97.79 0)
       (effects
@@
       )
     )
-    (property "Footprint" ""
+    (property "Footprint" "RoyalNode:U4_LTC4365_TSOT23_8_RC"
       (at 149.86 137.16 0)
       (effects
@@
       )
     )
-    (property "Footprint" ""
+    (property "Footprint" "RoyalNode:Q_POWER_INFINEON_PG_DSO_8_27_RC"
       (at 248.92 149.86 0)
       (effects
@@
       )
     )
-    (property "Footprint" ""
+    (property "Footprint" "RoyalNode:Q_POWER_INFINEON_PG_DSO_8_27_RC"
       (at 248.92 195.58 0)
       (effects
@@
       )
     )
-    (property "Footprint" ""
+    (property "Footprint" "RoyalNode:Q_POWER_INFINEON_PG_DSO_8_27_RC"
       (at 248.92 241.30 0)
       (effects
@@
       )
     )
-    (property "Footprint" ""
+    (property "Footprint" "RoyalNode:J_POWER_XT30PW_M_C431092_RC"
       (at 55.88 204.47 0)
       (effects
@@
       )
     )
-    (property "Footprint" ""
+    (property "Footprint" "RoyalNode:J_POWER_XT30PW_M_C431092_RC"
       (at 55.88 233.68 0)
       (effects
@@
       )
     )
-    (property "Footprint" ""
+    (property "Footprint" "RoyalNode:L1_COILCRAFT_XAL7070_222MEC_RC"
       (at 149.86 170.18 0)
       (effects
@@
       )
     )
-    (property "Footprint" ""
+    (property "Footprint" "RoyalNode:L2_COILCRAFT_XAL7030_222MEC_RC"
       (at 248.92 124.46 0)
       (effects

Commit message: Assign passive schematic footprints
Parts:
- C200, C201, C202, C203, C204, C205, C206, C207, C208, C209, C210, C211: footprint (none) -> Capacitor_SMD:C_1206_3216Metric
- C212, C213, C214, C216, C217, C218, C404, C406, C407, C408: footprint (none) -> Capacitor_SMD:C_0603_1608Metric
- C215, C405, C502: footprint (none) -> Capacitor_SMD:C_0805_2012Metric
- C400, C401, C402, C403, C500, C501: footprint (none) -> Capacitor_SMD:C_1210_3225Metric
- D1: footprint (none) -> LED_SMD:LED_0603_1608Metric
- R100, R101, R102, R103, R200, R201, R202, R203, R204, R205, R206, R207, R400, R401, R402, R403, R404, R405: footprint (none) -> Resistor_SMD:R_0603_1608Metric
Changed lines of the file:
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@@
       )
     )
-    (property "Footprint" ""
+    (property "Footprint" "Resistor_SMD:R_0603_1608Metric"
       (at 335.28 35.56 0)
       (effects
@@
       )
     )
-    (property "Footprint" ""
+    (property "Footprint" "Resistor_SMD:R_0603_1608Metric"
       (at 335.28 43.18 0)
       (effects
@@
       )
     )
-    (property "Footprint" ""
+    (property "Footprint" "Resistor_SMD:R_0603_1608Metric"
       (at 335.28 50.80 0)
       (effects
@@
       )
     )
-    (property "Footprint" ""
+    (property "Footprint" "Resistor_SMD:R_0603_1608Metric"
       (at 335.28 58.42 0)
       (effects
@@
       )
     )
-    (property "Footprint" ""
+    (property "Footprint" "Capacitor_SMD:C_1206_3216Metric"
       (at 335.28 66.04 0)
       (effects
@@
       )
     )
-    (property "Footprint" ""
+    (property "Footprint" "Capacitor_SMD:C_1206_3216Metric"
       (at 335.28 73.66 0)
       (effects
@@
       )
     )
-    (property "Footprint" ""
+    (property "Footprint" "Capacitor_SMD:C_1206_3216Metric"
       (at 335.28 81.28 0)
       (effects
@@
       )
     )
-    (property "Footprint" ""
+    (property "Footprint" "Capacitor_SMD:C_1206_3216Metric"
       (at 335.28 88.90 0)
       (effects
@@
       )
     )
-    (property "Footprint" ""
+    (property "Footprint" "Capacitor_SMD:C_1206_3216Metric"
       (at 335.28 96.52 0)
       (effects
@@
       )
     )
-    (property "Footprint" ""
+    (property "Footprint" "Capacitor_SMD:C_1206_3216Metric"
       (at 335.28 104.14 0)
       (effects
@@
       )
     )
-    (property "Footprint" ""
+    (property "Footprint" "Capacitor_SMD:C_1206_3216Metric"
       (at 335.28 111.76 0)
       (effects
@@
       )
     )
-    (property "Footprint" ""
+    (property "Footprint" "Capacitor_SMD:C_1206_3216Metric"
       (at 335.28 119.38 0)
       (effects
@@
       )
     )
-    (property "Footprint" ""
+    (property "Footprint" "Capacitor_SMD:C_1206_3216Metric"
       (at 335.28 127.00 0)
       (effects
@@
       )
     )
-    (property "Footprint" ""
+    (property "Footprint" "Capacitor_SMD:C_1206_3216Metric"
       (at 335.28 134.62 0)
       (effects
@@
       )
     )
-    (property "Footprint" ""
+    (property "Footprint" "Capacitor_SMD:C_1206_3216Metric"
       (at 335.28 142.24 0)
       (effects
@@
       )
     )
-    (property "Footprint" ""
+    (property "Footprint" "Capacitor_SMD:C_1206_3216Metric"
       (at 335.28 149.86 0)
       (effects
@@
       )
     )
-    (property "Footprint" ""
+    (property "Footprint" "Capacitor_SMD:C_0603_1608Metric"
       (at 335.28 157.48 0)
       (effects
@@
       )
     )
-    (property "Footprint" ""
+    (property "Footprint" "Capacitor_SMD:C_0603_1608Metric"
       (at 335.28 165.10 0)
       (effects
@@
       )
     )
-    (property "Footprint" ""
+    (property "Footprint" "Capacitor_SMD:C_0603_1608Metric"
       (at 335.28 172.72 0)
       (effects
@@
       )
     )
-    (property "Footprint" ""
+    (property "Footprint" "Capacitor_SMD:C_0805_2012Metric"
       (at 335.28 180.34 0)
       (effects
@@
       )
     )
-    (property "Footprint" ""
+    (property "Footprint" "Capacitor_SMD:C_0603_1608Metric"
       (at 335.28 187.96 0)
       (effects
@@
       )
     )
-    (property "Footprint" ""
+    (property "Footprint" "Capacitor_SMD:C_0603_1608Metric"
       (at 335.28 195.58 0)
       (effects
@@
       )
     )
-    (property "Footprint" ""
+    (property "Footprint" "Capacitor_SMD:C_0603_1608Metric"
       (at 386.08 35.56 0)
       (effects
@@
       )
     )
-    (property "Footprint" ""
+    (property "Footprint" "Resistor_SMD:R_0603_1608Metric"
       (at 386.08 43.18 0)
       (effects
@@
       )
     )
-    (property "Footprint" ""
+    (property "Footprint" "Resistor_SMD:R_0603_1608Metric"
       (at 386.08 50.80 0)
       (effects
@@
       )
     )
-    (property "Footprint" ""
+    (property "Footprint" "Resistor_SMD:R_0603_1608Metric"
       (at 386.08 58.42 0)
       (effects
@@
       )
     )
-    (property "Footprint" ""
+    (property "Footprint" "Resistor_SMD:R_0603_1608Metric"
       (at 386.08 66.04 0)
       (effects
@@
       )
     )
-    (property "Footprint" ""
+    (property "Footprint" "Resistor_SMD:R_0603_1608Metric"
       (at 386.08 73.66 0)
       (effects
@@
       )
     )
-    (property "Footprint" ""
+    (property "Footprint" "Resistor_SMD:R_0603_1608Metric"
       (at 386.08 81.28 0)
       (effects
@@
       )
     )
-    (property "Footprint" ""
+    (property "Footprint" "Resistor_SMD:R_0603_1608Metric"
       (at 386.08 88.90 0)
       (effects
@@
       )
     )
-    (property "Footprint" ""
+    (property "Footprint" "LED_SMD:LED_0603_1608Metric"
       (at 386.08 96.52 0)
       (effects
@@
       )
     )
-    (property "Footprint" ""
+    (property "Footprint" "Resistor_SMD:R_0603_1608Metric"
       (at 386.08 104.14 0)
       (effects
@@
       )
     )
-    (property "Footprint" ""
+    (property "Footprint" "Capacitor_SMD:C_1210_3225Metric"
       (at 386.08 111.76 0)
       (effects
@@
       )
     )
-    (property "Footprint" ""
+    (property "Footprint" "Capacitor_SMD:C_1210_3225Metric"
       (at 386.08 119.38 0)
       (effects
@@
       )
     )
-    (property "Footprint" ""
+    (property "Footprint" "Capacitor_SMD:C_1210_3225Metric"
       (at 386.08 127.00 0)
       (effects
@@
       )
     )
-    (property "Footprint" ""
+    (property "Footprint" "Capacitor_SMD:C_1210_3225Metric"
       (at 386.08 134.62 0)
       (effects
@@
       )
     )
-    (property "Footprint" ""
+    (property "Footprint" "Capacitor_SMD:C_0603_1608Metric"
       (at 386.08 142.24 0)
       (effects
@@
       )
     )
-    (property "Footprint" ""
+    (property "Footprint" "Capacitor_SMD:C_0805_2012Metric"
       (at 386.08 149.86 0)
       (effects
@@
       )
     )
-    (property "Footprint" ""
+    (property "Footprint" "Capacitor_SMD:C_0603_1608Metric"
       (at 386.08 157.48 0)
       (effects
@@
       )
     )
-    (property "Footprint" ""
+    (property "Footprint" "Capacitor_SMD:C_0603_1608Metric"
       (at 386.08 165.10 0)
       (effects
@@
       )
     )
-    (property "Footprint" ""
+    (property "Footprint" "Capacitor_SMD:C_0603_1608Metric"
       (at 386.08 172.72 0)
       (effects
@@
       )
     )
-    (property "Footprint" ""
+    (property "Footprint" "Resistor_SMD:R_0603_1608Metric"
       (at 386.08 180.34 0)
       (effects
@@
       )
     )
-    (property "Footprint" ""
+    (property "Footprint" "Resistor_SMD:R_0603_1608Metric"
       (at 386.08 187.96 0)
       (effects
@@
       )
     )
-    (property "Footprint" ""
+    (property "Footprint" "Resistor_SMD:R_0603_1608Metric"
       (at 386.08 195.58 0)
       (effects
@@
       )
     )
-    (property "Footprint" ""
+    (property "Footprint" "Resistor_SMD:R_0603_1608Metric"
       (at 436.88 35.56 0)
       (effects
@@
       )
     )
-    (property "Footprint" ""
+    (property "Footprint" "Resistor_SMD:R_0603_1608Metric"
       (at 436.88 43.18 0)
       (effects
@@
       )
     )
-    (property "Footprint" ""
+    (property "Footprint" "Resistor_SMD:R_0603_1608Metric"
       (at 436.88 50.80 0)
       (effects
@@
       )
     )
-    (property "Footprint" ""
+    (property "Footprint" "Capacitor_SMD:C_1210_3225Metric"
       (at 436.88 58.42 0)
       (effects
@@
       )
     )
-    (property "Footprint" ""
+    (property "Footprint" "Capacitor_SMD:C_1210_3225Metric"
       (at 436.88 66.04 0)
       (effects
@@
       )
     )
-    (property "Footprint" ""
+    (property "Footprint" "Capacitor_SMD:C_0805_2012Metric"
       (at 436.88 73.66 0)
       (effects

Commit message: Standardize low-current connectors on JST-GH
Parts:
- J3: value XIAO BAT HARNESS -> JST-GH XIAO BAT HARNESS; footprint (none) -> RoyalNode:J_LOW_JST_GH_SM02B_GHS_TB_RC; symbol RoyalNode:RN_JST_PH_2 -> RoyalNode:RN_JST_GH_2
- J4: value BATTERY NTC -> JST-GH BATTERY NTC; footprint (none) -> RoyalNode:J_LOW_JST_GH_SM02B_GHS_TB_RC; symbol RoyalNode:RN_JST_PH_2 -> RoyalNode:RN_JST_GH_2
Changed lines of the file:
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@@
   )
   (symbol
-    (lib_id "RoyalNode:RN_JST_PH_2")
+    (lib_id "RoyalNode:RN_JST_GH_2")
     (at 149.86 204.47 0)
     (unit 1)
@@
       )
     )
-    (property "Value" "XIAO BAT HARNESS"
+    (property "Value" "JST-GH XIAO BAT HARNESS"
       (at 149.86 228.47 0)
       (effects
@@
       )
     )
-    (property "Footprint" ""
+    (property "Footprint" "RoyalNode:J_LOW_JST_GH_SM02B_GHS_TB_RC"
       (at 149.86 204.47 0)
       (effects
@@
   )
   (symbol
-    (lib_id "RoyalNode:RN_JST_PH_2")
+    (lib_id "RoyalNode:RN_JST_GH_2")
     (at 149.86 233.68 0)
     (unit 1)
@@
       )
     )
-    (property "Value" "BATTERY NTC"
+    (property "Value" "JST-GH BATTERY NTC"
       (at 149.86 257.68 0)
       (effects
@@
       )
     )
-    (property "Footprint" ""
+    (property "Footprint" "RoyalNode:J_LOW_JST_GH_SM02B_GHS_TB_RC"
       (at 149.86 233.68 0)
       (effects

Commit message: Assign solar fuse footprint
Parts:
- F1: footprint (none) -> RoyalNode:F1_LITTELFUSE_483_1206_RC
Changed lines of the file:
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@@
       )
     )
-    (property "Footprint" ""
+    (property "Footprint" "RoyalNode:F1_LITTELFUSE_483_1206_RC"
       (at 55.88 184.15 0)
       (effects

Commit message: Assign E22 bulk capacitor footprint
Parts:
- C503: footprint (none) -> RoyalNode:C503_PANASONIC_10SVPC330M_8X6P9_RC
Changed lines of the file:
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@@
       )
     )
-    (property "Footprint" ""
+    (property "Footprint" "RoyalNode:C503_PANASONIC_10SVPC330M_8X6P9_RC"
       (at 436.88 81.28 0)
       (effects
